Commit message: added rgb-d camera definitions do xacro/urdf for the base camera and an elevated one

File: robutler_description/turtlebot3_waffle_pi.gazebo.xacro (robot description, xacro)
@@ -136,20 +136,24 @@
 <!--link : https://www.raspberrypi.org/documentation/hardware/camera/-->
   <gazebo reference="camera_rgb_frame">
-    <sensor type="camera" name="Pi Camera">
+    <sensor type="depth" name="camera">
       <always_on>true</always_on>
       <visualize>$(arg camera_visual)</visualize>
       <camera>
-          <horizontal_fov>1.085595</horizontal_fov>
-          <image>
-              <width>640</width>
-              <height>480</height>
-              <format>R8G8B8</format>
-          </image>
-          <clip>
-              <near>0.03</near>
-              <far>100</far>
-          </clip>
+        <horizontal_fov>1.047198</horizontal_fov>
+        <image>
+          <width>640</width>
+          <height>480</height>
+          <format>B8G8R8</format>
+        </image>
+        <clip>
+          <near>0.05</near>
+          <far>3.0</far>
+        </clip>
+        <depth_camera>
+          <output>depths</output>
+        </depth_camera>
       </camera>
-      <plugin name="camera_controller" filename="libgazebo_ros_camera.so">
+      <plugin name="camera_controller" filename="libgazebo_ros_openni_kinect.so">
+        <baseline>0.2</baseline>
         <alwaysOn>true</alwaysOn>
         <updateRate>30.0</updateRate>
@@ -158,12 +162,45 @@
         <imageTopicName>rgb/image_raw</imageTopicName>
         <cameraInfoTopicName>rgb/camera_info</cameraInfoTopicName>
-        <hackBaseline>0.07</hackBaseline>
-        <distortionK1>0.0</distortionK1>
-        <distortionK2>0.0</distortionK2>
-        <distortionK3>0.0</distortionK3>
-        <distortionT1>0.0</distortionT1>
-        <distortionT2>0.0</distortionT2>
+        <depthImageTopicName>depth/image_raw</depthImageTopicName>
+        <depthImageInfoTopicName>depth/camera_info</depthImageInfoTopicName>
+        <pointCloudTopicName>depth/points</pointCloudTopicName>
+        <depthImageCameraInfoTopicName>depth/camera_info</depthImageCameraInfoTopicName>
       </plugin>
     </sensor>
   </gazebo>
+  <!-- Elevated RGB-D Camera -->
+  <gazebo reference="elevated_camera_rgb_frame">
+    <sensor type="depth" name="elevated_camera">
+      <always_on>true</always_on>
+      <visualize>$(arg camera_visual)</visualize>
+      <camera>
+        <horizontal_fov>1.047198</horizontal_fov>
+        <image>
+          <width>640</width>
+          <height>480</height>
+          <format>B8G8R8</format>
+        </image>
+        <clip>
+          <near>0.05</near>
+          <far>3.0</far>
+        </clip>
+        <depth_camera>
+          <output>depths</output>
+        </depth_camera>
+      </camera>
+      <plugin name="elevated_camera_controller" filename="libgazebo_ros_openni_kinect.so">
+        <baseline>0.2</baseline>
+        <alwaysOn>true</alwaysOn>
+        <updateRate>30.0</updateRate>
+        <cameraName>elevated_camera</cameraName>
+        <frameName>elevated_camera_rgb_optical_frame</frameName>
+        <imageTopicName>rgb/image_raw</imageTopicName>
+        <cameraInfoTopicName>rgb/camera_info</cameraInfoTopicName>
+        <depthImageTopicName>depth/image_raw</depthImageTopicName>
+        <depthImageInfoTopicName>depth/camera_info</depthImageInfoTopicName>
+        <pointCloudTopicName>depth/points</pointCloudTopicName>
+        <depthImageCameraInfoTopicName>depth/camera_info</depthImageCameraInfoTopicName>
+      </plugin>
+    </sensor>
+  </gazebo>
 </robot>

File: robutler_description/turtlebot3_waffle_pi.urdf.xacro (robot description, xacro)
@@ -166,10 +166,21 @@
   </joint>
   <link name="camera_link">
-    <collision>
+    <visual>
       <origin xyz="0.005 0.011 0.013" rpy="0 0 0"/>
       <geometry>
-        <box size="0.015 0.030 0.027"/>
-      </geometry>
-    </collision>
+        <box size="0.025 0.035 0.027"/>
+      </geometry>
+      <material name="dark"/>
+    </visual>
+    <collision>
+      <origin xyz="0.005 0.011 0.013" rpy="0 0 0"/>
+      <geometry>
+        <box size="0.025 0.035 0.027"/>
+      </geometry>
+    </collision>
+    <inertial>
+      <mass value="0.01"/>
+      <inertia ixx="0.001" ixy="0" ixz="0" iyy="0.001" iyz="0" izz="0.001"/>
+    </inertial>
   </link>
   <joint name="camera_rgb_joint" type="fixed">
@@ -185,3 +196,85 @@
   </joint>
   <link name="camera_rgb_optical_frame"/>
+  <!-- Elevated Camera Assembly -->
+  <joint name="camera_pole_joint" type="fixed">
+    <parent link="base_link"/>
+    <child link="camera_pole"/>
+    <origin xyz="-0.064 0 0.094" rpy="0 0 0"/>
+  </joint>
+  <link name="camera_pole">
+    <visual>
+      <origin xyz="0 0 0.4" rpy="0 0 0"/>
+      <geometry>
+        <cylinder length="0.8" radius="0.008"/>
+      </geometry>
+      <material name="grey"/>
+    </visual>
+    <collision>
+      <origin xyz="0 0 0.4" rpy="0 0 0"/>
+      <geometry>
+        <cylinder length="0.8" radius="0.008"/>
+      </geometry>
+    </collision>
+    <inertial>
+      <origin xyz="0 0 0.4" rpy="0 0 0"/>
+      <mass value="0.2"/>
+      <inertia ixx="0.002" ixy="0" ixz="0" iyy="0.002" iyz="0" izz="0.001"/>
+    </inertial>
+  </link>
+  <joint name="elevated_camera_base_joint" type="fixed">
+    <parent link="camera_pole"/>
+    <child link="elevated_camera_base"/>
+    <origin xyz="0 0 0.8" rpy="0 0 0"/>
+  </joint>
+  <link name="elevated_camera_base">
+    <visual>
+      <geometry>
+        <box size="0.03 0.03 0.01"/>
+      </geometry>
+      <material name="dark"/>
+    </visual>
+    <collision>
+      <geometry>
+        <box size="0.03 0.03 0.01"/>
+      </geometry>
+    </collision>
+    <inertial>
+      <mass value="0.01"/>
+      <inertia ixx="0.001" ixy="0" ixz="0" iyy="0.001" iyz="0" izz="0.001"/>
+    </inertial>
+  </link>
+  <joint name="elevated_camera_joint" type="fixed">
+    <parent link="elevated_camera_base"/>
+    <child link="elevated_camera_link"/>
+    <origin xyz="0.015 0 0.0135" rpy="0 0 0"/>
+  </joint>
+  <link name="elevated_camera_link">
+    <visual>
+      <geometry>
+        <box size="0.025 0.035 0.027"/>
+      </geometry>
+      <material name="dark"/>
+    </visual>
+    <collision>
+      <geometry>
+        <box size="0.025 0.035 0.027"/>
+      </geometry>
+    </collision>
+    <inertial>
+      <mass value="0.01"/>
+      <inertia ixx="0.001" ixy="0" ixz="0" iyy="0.001" iyz="0" izz="0.001"/>
+    </inertial>
+  </link>
+  <joint name="elevated_camera_rgb_joint" type="fixed">
+    <origin xyz="0.003 0.011 0.009" rpy="0 0 0"/>
+    <parent link="elevated_camera_link"/>
+    <child link="elevated_camera_rgb_frame"/>
+  </joint>
+  <link name="elevated_camera_rgb_frame"/>
+  <joint name="elevated_camera_rgb_optical_joint" type="fixed">
+    <origin xyz="0 0 0" rpy="-1.57 0 -1.57"/>
+    <parent link="elevated_camera_rgb_frame"/>
+    <child link="elevated_camera_rgb_optical_frame"/>
+  </joint>
+  <link name="elevated_camera_rgb_optical_frame"/>
 </robot>
